File: HW/TP_STM32L021K4T6/TP_STM32L021K4T6.kicad_pcb (KiCad board)
At the start: 2 copper layers, 58.5 x 48.5 mm, 27 parts, among them J1 Conn_02x07_Odd_Even, U1 STM32L021K4Tx, U2 BU33SD5WG-TR, U3 MCP4801-EMC

Commit message: firware
Parts:
- D1, D2: footprint LED_SMD:LED_0201_0603Metric_Pad0.64x0.40mm_HandSolder -> LED_SMD:LED_0603_1608Metric_Pad1.05x0.95mm_HandSolder
- Input1, Output1, Power1: footprint Connector_JST:JST_XH_B2B-XH-AM_1x02_P2.50mm_Vertical -> Connector_JST:JST_XH_B2B-XH-A_1x02_P2.50mm_Vertical
- U3: footprint Package_DFN_QFN:DFN-8-1EP_3x2mm_P0.5mm_EP1.75x1.45mm -> Package_SO:SOIC-8_3.9x4.9mm_P1.27mm
- moved C3 37.0 mm to (110.4, 86.5), turned to -90 degrees
- moved C2 25.7 mm to (117.2, 72.3)
- moved C8 25.0 mm to (117.0, 62.3)
- moved C10 23.4 mm to (122.1, 88.4)
- moved C9 19.4 mm to (121.1, 78.4), turned to 180 degrees
- moved C4 13.2 mm to (108.3, 86.5), turned to -90 degrees
- moved R2 3.99 mm to (106.3, 86.6)
- moved Input1 3.57 mm to (93.2, 75.0), turned to -90 degrees
- moved D1 2.95 mm to (113.5, 69.0), turned to 180 degrees
- moved U3 2.95 mm to (121.9, 83.6), turned to -90 degrees
- moved Power1 2.39 mm to (112.0, 57.2), turned to 180 degrees
- moved C5 1.28 mm to (121.3, 72.3)
- moved L1 1.28 mm to (121.1, 74.3)
- moved C6 1.28 mm to (121.1, 76.3)
- moved C7 1.01 mm to (109.5, 63.1)
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Routing:
- net +3V3: track 0.00 -> 66.3 mm
- net NRST: track 0.00 -> 50.3 mm, vias 0 -> 2
- net USART2_RX: track 0.00 -> 38.4 mm, vias 0 -> 2
- net USART2_TX: track 0.00 -> 36.5 mm, vias 0 -> 2
- net ADC_IN1: track 0.00 -> 35.6 mm
- net +3.3VA: track 0.00 -> 28.9 mm, vias 0 -> 2
- net GND: track 0.00 -> 27.5 mm, vias 0 -> 8
- net SWDIO: track 0.00 -> 26.7 mm, vias 0 -> 2
- net SWDCLK: track 0.00 -> 26.7 mm, vias 0 -> 2
- net DAC_OUT: track 0.00 -> 22.3 mm
- net +5V: track 0.00 -> 11.8 mm
- net DAC_nCS: track 0.00 -> 8.80 mm
- net SPI1_SCK: track 0.00 -> 7.32 mm
- net Net-(U1-PB9): track 0.00 -> 6.55 mm
- net LED_STATUS: track 0.00 -> 6.42 mm
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